File: hardware/IFB-40002-R02 - I2C_Joystick.brd (EAGLE design)
At the start: 30 x 30 mm, 26 parts, among them J3 CUTTABLE_JUMPER, J4 CUT_JUMPER_2X, U3 ATTINY841-MMHR

Commit message: updated hardware files
Parts:
- removed J3: CUTTABLE_JUMPER, PlayingWithFusion_Breakout-Lib:SMT_CUTTABLE_JUMPER
- added C3, C4: 0.1uF, rcl:C0603K
- added J5: CUT_JUMPER_2X, PlayingWithFusion_Breakout-Lib:SMT_2X_CUTTABLE_JUMPER
- added R5: 100k, rcl:R0603
- J1, J2: value (none) -> QWIICSIDE; device SparkFun-Connectors:1X04_1MM_RA -> PlayingWithFusion_JST:SM04B-SRSS-TB
- moved SO1 25.5 mm to (2.25, 2.25), turned to 270 degrees
- moved SO2 25.5 mm to (27.8, 27.8), turned to 270 degrees
- moved SO3 25.5 mm to (27.8, 2.25), turned to 270 degrees
- moved SO4 25.5 mm to (2.25, 27.8), turned to 270 degrees
- moved U$3 22.7 mm to (6.40, 27.6), turned to 270 degrees
- moved U$2 22.6 mm to (27.6, 5.21), turned to 270 degrees
- moved VCC 21.6 mm to (23.0, 2.00), turned to 270 degrees
- moved LOGO1 20.2 mm to (26.8, 23.0), turned to 270 degrees
- moved LOGO2 20.2 mm to (26.8, 7.04), turned to 90 degrees
- moved GND 19.9 mm to (20.5, 2.00), turned to 270 degrees
- moved RST 19.5 mm to (10.3, 2.00), turned to 270 degrees
- moved MOSI 18.8 mm to (17.9, 2.00), turned to 270 degrees
- moved SCK 18.6 mm to (12.8, 2.00), turned to 270 degrees
- moved MISO 18.4 mm to (15.4, 2.00), turned to 270 degrees
- moved J1 15.8 mm to (5.25, 11.0), turned to 90 degrees
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Connections:
- removed net N$1: J3.2, R4.2, U3.15
- new net ADDR0: J5.3, R4.2, U3.15
- new net ADDR1: J5.1, R5.2, U3.14
- net GND: now also C3.2, C4.2, J5.2; no longer J3.1
- net VCC: now also C3.1, C4.1, R5.1
Routing:
- net ADDR0: track 0.00 -> 8.66 mm
- net N$1: track 7.71 -> 0.00 mm
- net VCC: track 83.7 -> 76.2 mm, vias 0 -> 2
- net ADDR1: track 0.00 -> 6.92 mm
- net SCL: track 42.0 -> 36.8 mm
- net GND: track 5.64 -> 8.61 mm, vias 14 -> 16
- net JH: track 12.2 -> 14.4 mm
- net SDA: track 36.2 -> 34.7 mm
- net N$3: track 3.19 -> 2.39 mm
- net SEL: track 14.7 -> 15.4 mm, vias 2 -> 0
- net N$2: track 5.51 -> 4.85 mm
Other:
- board text added: "0 1"
- board text added: "C3"
- board text added: "C4"
- board text added: "R5"
