File: hardware/IFB-40002-R02 - I2C_Joystick.sch (EAGLE design)
At the start: 26 parts, among them J3 CUTTABLE_JUMPER, J4 CUT_JUMPER_2X, U3 ATTINY841-MMHR

Commit message: updated hardware files
Parts:
- removed J3: CUTTABLE_JUMPER, PlayingWithFusion_Breakout-Lib:CUTTABLE_JUMPER
- added C3, C4: 0.1uF, rcl:C-USC0603K
- added J5: CUT_JUMPER_2X, PlayingWithFusion_Breakout-Lib:CUT_JUMPER_2X
- added R5: 100k, rcl:R-US_R0603
- J1, J2: value (none) -> QWIICSIDE; device SparkFun-Connectors:QWIIC_CONNECTORJS-1MM -> PlayingWithFusion_JST:QWIICSIDE
Connections:
- removed net N$1: J3.2, R4.2, U3.PA7
- new net ADDR0: J5.3, R4.2, U3.PA7
- new net ADDR1: J5.1, R5.2, U3.PB2
- net GND: now also C3.2, C4.2, J1.1, J2.1, J5.2; no longer J1.GND, J2.GND, J3.1
- net SCL: now also J1.4, J2.4; no longer J1.SCL, J2.SCL
- net SDA: now also J1.3, J2.3; no longer J1.SDA, J2.SDA
- net VCC: now also C3.1, C4.1, J1.2, J2.2, R5.1; no longer J1.VCC, J2.VCC
Other:
- moved on the sheet: C1, C2, J4, R1, R3, R4
